File: Hardware/PCA9306_Breakout.brd (EAGLE design)
At the start: 19.1 x 12.7 mm, 39 parts, among them U1 PCA9306

Commit message: Changes version number to v20
Other:
- board text added: "v20"
- board text removed: "v15"
Changed lines of the file:
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@@
 <wire x1="19.05" y1="12.7" x2="0" y2="12.7" width="0.2032" layer="20"/>
 <wire x1="0" y1="12.7" x2="0" y2="0" width="0.2032" layer="20"/>
-<text x="6.0452" y="0.2794" size="0.8128" layer="16" font="vector" ratio="12" rot="MR0">v15</text>
+<text x="6.0452" y="0.2794" size="0.8128" layer="16" font="vector" ratio="12" rot="MR0">v20</text>
 <text x="25.4" y="-10.16" size="1.778" layer="27" font="vector" ratio="15">T. Klopfenstein</text>
 <dimension x1="0" y1="12.7" x2="19.05" y2="12.7" x3="9.525" y3="13.97" textsize="1.778" layer="47" unit="inch"/>
