File: Hardware/PCA9306_Breakout.sch (EAGLE design)
At the start: 18 parts, among them U1 PCA9306

Commit message: Changes version number to v20
Other:
- note added: "v20"
- note removed: "v15"
Changed lines of the file:
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@@
 <plain>
 <text x="166.37" y="11.684" size="2.54" layer="94" font="vector">T. Klopfenstein</text>
-<text x="238.76" y="7.62" size="2.54" layer="94" font="vector">v15</text>
+<text x="238.76" y="7.62" size="2.54" layer="94" font="vector">v20</text>
 <wire x1="121.92" y1="185.42" x2="121.92" y2="0" width="0.2032" layer="97" style="shortdash"/>
 <text x="7.62" y="175.26" size="2.54" layer="94" font="vector">Logic Level Translator PCA9306</text>
