File: Hardware/SparkFun_Level_Translator_PCA9306.brd (EAGLE design)
At the start: 19.1 x 12.7 mm, 39 parts, among them U1 PCA9306

Commit message: Adds production files
Parts:
- removed U$16: (no value), Jumper_Options:SWCH0
- added U$1: (no value), Jumper_Options:SWITCH1
